File: macropad-v1.kicad_pcb (KiCad board)
At the start: 2 copper layers, 72.2 x 38.1 mm, 24 parts, among them SW1 SW_Push, U1 ATmega32U4-AU, Y1 16MHz

Commit message: pcb routes
Parts:
- F1, R2, R3, SW1: moved to B.Cu
- moved R2 189.6 mm to (57.1, 108.0), turned to 90 degrees
- moved R3 174.2 mm to (59.5, 108.0), turned to 90 degrees
- moved R4 156.2 mm to (78.6, 108.7)
- moved SW1 144.4 mm to (81.0, 117.5)
- moved F1 135.4 mm to (83.3, 99.2), turned to 90 degrees
- moved C7 24.7 mm to (83.3, 104.0), turned to 270 degrees
- moved R1 5.42 mm to (60.3, 99.2)
Connections:
- U1 pad 29: Net-(U1-Pad29) -> ROW0
- U1 pad 30: Net-(U1-Pad30) -> COL1
- U1 pad 31: Net-(U1-Pad31) -> COL0
- U1 pad 32: Net-(U1-Pad32) -> ROW1
Routing:
- net GND: track 0.00 -> 117.9 mm
- net +5V: track 0.00 -> 81.7 mm, vias 0 -> 8
- net COL1: track 0.00 -> 58.4 mm
- net ROW0: track 0.00 -> 54.3 mm
- net ROW1: track 0.00 -> 53.2 mm
- net Net-(R1-Pad2): track 0.00 -> 52.2 mm, vias 0 -> 2
- net D+: track 0.00 -> 41.1 mm
- net D-: track 0.00 -> 39.8 mm
- net COL0: track 0.00 -> 38.2 mm
- net Net-(USB1-Pad6): track 0.00 -> 16.3 mm
- net Net-(C2-Pad1): track 0.00 -> 10.3 mm
- net VCC: track 0.00 -> 9.24 mm
- net Net-(R2-Pad1): track 0.00 -> 8.97 mm
- net Net-(C1-Pad1): track 0.00 -> 8.08 mm
- net Net-(D2-Pad2): track 0.00 -> 6.62 mm
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Other:
- net class Default: trace_width 0.25 -> 0.254
- net class Power added: clearance 0.2, trace_width 0.381, via_dia 0.8, via_drill 0.4

Commit message: gerber
Connections:
- USB1 pad 6: Net-(USB1-Pad6) -> GND
Routing:
- net Net-(USB1-Pad6): track 16.3 -> 0.00 mm
- net GND: track 117.9 -> 126.6 mm
- added copper zone on B.Cu, net GND
Other:
- board text added: "Four-Key MacroPad"
Changed lines of the file:
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@@
   (general
     (thickness 1.6)
-    (drawings 8)
-    (tracks 191)
+    (drawings 9)
+    (tracks 194)
     (zones 0)
     (modules 24)
-    (nets 45)
+    (nets 44)
   )
   (page A4)
@@
   (net 41 "Net-(U1-Pad8)")
   (net 42 "Net-(U1-Pad1)")
-  (net 43 "Net-(USB1-Pad6)")
-  (net 44 "Net-(USB1-Pad2)")
+  (net 43 "Net-(USB1-Pad2)")
   (net_class Default "This is the default net class."
     (clearance 0.2)
@@
     (add_net "Net-(U1-Pad9)")
     (add_net "Net-(USB1-Pad2)")
-    (add_net "Net-(USB1-Pad6)")
     (add_net ROW0)
     (add_net ROW1)
@@
     (fp_line (start 3.25 1.25) (end 5.5 1.25) (layer B.CrtYd) (width 0.15))
     (pad 6 thru_hole oval (at 0 3.65 270) (size 2.7 1.7) (drill oval 1.9 0.7) (layers *.Cu *.Mask)
-      (net 43 "Net-(USB1-Pad6)"))
+      (net 1 GND))
     (pad 6 thru_hole oval (at 0 -3.65 270) (size 2.7 1.7) (drill oval 1.9 0.7) (layers *.Cu *.Mask)
-      (net 43 "Net-(USB1-Pad6)"))
+      (net 1 GND))
     (pad 6 thru_hole oval (at 4.5 -3.65 270) (size 2.7 1.7) (drill oval 1.9 0.7) (layers *.Cu *.Mask)
-      (net 43 "Net-(USB1-Pad6)"))
+      (net 1 GND))
     (pad 6 thru_hole oval (at 4.5 3.65 270) (size 2.7 1.7) (drill oval 1.9 0.7) (layers *.Cu *.Mask)
-      (net 43 "Net-(USB1-Pad6)"))
+      (net 1 GND))
     (pad 5 smd rect (at 4.5 1.6 270) (size 2.25 0.5) (layers B.Cu B.Paste B.Mask)
       (net 12 VCC))
@@
       (net 16 D+))
     (pad 2 smd rect (at 4.5 -0.8 270) (size 2.25 0.5) (layers B.Cu B.Paste B.Mask)
-      (net 44 "Net-(USB1-Pad2)"))
+      (net 43 "Net-(USB1-Pad2)"))
     (pad 1 smd rect (at 4.5 -1.6 270) (size 2.25 0.5) (layers B.Cu B.Paste B.Mask)
       (net 1 GND))
@@
     (tags SOD-123)
     (attr smd)
-    (fp_text reference D4 (at 0 2 90) (layer B.SilkS)
+    (fp_text reference D4 (at -3.96875 0 90) (layer B.SilkS)
       (effects (font (size 1 1) (thickness 0.15)) (justify mirror))
     )
@@
     (tags SOD-123)
     (attr smd)
-    (fp_text reference D2 (at 0 2 90) (layer B.SilkS)
+    (fp_text reference D2 (at -3.96875 0 90) (layer B.SilkS)
       (effects (font (size 1 1) (thickness 0.15)) (justify mirror))
     )
@@
       (rotate (xyz 0 0 0))
     )
+  )
+  (gr_text "Four-Key MacroPad" (at 65.0875 86.51875) (layer F.SilkS)
+    (effects (font (size 1 1) (thickness 0.15)))
   )
   (gr_line (start 124.61875 86.51875) (end 124.61875 119.85625) (layer Edge.Cuts) (width 0.2))
@@
   (segment (start 75.34325 107.80625) (end 74.915 107.378) (width 0.254) (layer B.Cu) (net 20))
   (segment (start 78.58125 107.80625) (end 75.34325 107.80625) (width 0.254) (layer B.Cu) (net 20))
-  (segment (start 84.6125 85.725) (end 84.6125 90.225) (width 0.254) (layer F.Cu) (net 43))
-  (segment (start 84.6125 85.725) (end 77.3125 85.725) (width 0.254) (layer F.Cu) (net 43))
-  (segment (start 77.3125 85.725) (end 77.3125 90.225) (width 0.254) (layer F.Cu) (net 43))
+  (segment (start 77.3125 85.725) (end 79.375 85.725) (width 0.381) (layer B.Cu) (net 1))
+  (segment (start 84.6125 85.725) (end 82.55 85.725) (width 0.381) (layer B.Cu) (net 1))
+  (segment (start 84.6125 90.225) (end 84.6125 88.58125) (width 0.381) (layer B.Cu) (net 1))
+  (segment (start 84.6125 88.58125) (end 84.1375 88.10625) (width 0.381) (layer B.Cu) (net 1))
+  (segment (start 77.3125 90.225) (end 77.3125 90.9625) (width 0.381) (layer B.Cu) (net 1))
+  (segment (start 77.3125 90.9625) (end 76.2 92.075) (width 0.381) (layer B.Cu) (net 1))
+  (zone (net 1) (net_name GND) (layer B.Cu) (hatch edge 0.508)
+    (connect_pads (clearance 0.508))
+    (min_thickness 0.254)
+    (fill yes (arc_segments 32) (thermal_gap 0.508) (thermal_bridge_width 0.508))
+    (polygon
+      (pts
+        (xy 86.51875 122.2375) (xy 52.3875 122.2375) (xy 52.3875 84.1375) (xy 86.51875 84.1375)
+      )
+    )
+  )
 )
